File: Circuit/SlideBoard.brd (EAGLE design)
At the start: 19.1 x 77.5 mm, 24 parts

Commit message: Updated controller board to include BLE112 for easier soldering
Parts:
- R3: value 10k -> 50k
- U$1: value BLE113 -> BLE112; device Random:BLE113 -> temp:BLE112
- moved RESET 11.8 mm to (18.5, 36.3), turned to 0 degrees
- moved U$1 6.35 mm to (3.81, 19.1)
- moved UART 6.10 mm to (10.9, 34.8), turned to 180 degrees
- moved C1 4.94 mm to (12.4, 25.1), turned to 90 degrees
- moved -LED+ 3.94 mm to (18.5, 9.78)
- moved R4 3.87 mm to (18.5, 12.6)
- moved CAM 3.81 mm to (22.9, 43.9)
- moved YAW 3.81 mm to (22.9, 57.1)
- moved R3 3.14 mm to (14.8, 34.6), turned to 270 degrees
- moved PROG 2.54 mm to (11.4, 5.08)
- moved PWR 1.48 mm to (11.2, 14.0), turned to 45 degrees
- moved R6 1.48 mm to (11.9, 38.1)
- moved C2 0.80 mm to (5.21, 25.7), turned to 270 degrees
- moved C4 0.38 mm to (9.65, 24.6), turned to 90 degrees
Connections:
- net FOCUS: now also U$1.P17; no longer U$1.P$23
- net GND: now also U$1.P1, U$1.P10, U$1.P21, U$1.P30; no longer U$1.P$1, U$1.P$18, U$1.P$2, U$1.P$25, U$1.P$3, U$1.P$36, U$1.P$4, U$1.P$5, U$1.P$6, U$1.P$7
- net N$6: now also U$1.P15; no longer U$1.P$21
- net N$8: now also U$1.P14; no longer U$1.P$20
- net N$9: now also U$1.P19; no longer U$1.P$26
- net P2_1/PROG: now also U$1.P5; no longer U$1.P$10
- net P2_2/PROG: now also U$1.P4; no longer U$1.P$9
- net RESET: now also U$1.P29; no longer U$1.P$34
- net RX: now also U$1.P26; no longer U$1.P$31
- net SHUTTER: now also U$1.P18; no longer U$1.P$24
- net TX: now also U$1.P25; no longer U$1.P$30
- net VCC: now also U$1.P2, U$1.P20, U$1.P3; no longer U$1.P$17, U$1.P$8
- net YAW_LOW: now also U$1.P22; no longer U$1.P$27
Routing:
- net VCC: track 21.3 -> 45.4 mm, vias 5 -> 8
- net N$6: track 0.00 -> 16.7 mm
- net TX: track 13.5 -> 3.79 mm, vias 1 -> 0
- net N$8: track 0.00 -> 8.00 mm
- net RX: track 11.1 -> 4.24 mm, vias 1 -> 0
- net SHUTTER: track 18.7 -> 23.6 mm, vias 0 -> 2
- net GND: track 46.7 -> 42.5 mm, vias 7 -> 6
- net YAW_LOW: track 47.2 -> 43.2 mm
- net N$9: track 42.4 -> 46.2 mm
- net N$1: track 3.25 -> 6.63 mm
- net YAW: track 23.9 -> 26.3 mm
- net +5V: track 36.8 -> 34.4 mm
- net N$4: track 6.06 -> 8.34 mm
- net FOCUS: track 29.3 -> 31.5 mm, vias 2 -> 0
- net N$5: track 23.4 -> 25.0 mm
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Other:
- board size 19.1 x 77.5 mm -> 22.9 x 78.7 mm

Commit message: Fixed missing power connection
Routing:
- net N$9: track 46.2 -> 47.3 mm
Changed lines of the file:
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@@
 <setting verticaltext="up"/>
 </settings>
-<grid distance="0.05" unitdist="inch" unit="inch" style="lines" multiple="1" display="yes" altdistance="0.01" altunitdist="inch" altunit="inch"/>
+<grid distance="0.005" unitdist="inch" unit="inch" style="lines" multiple="1" display="yes" altdistance="0.01" altunitdist="inch" altunit="inch"/>
 <layers>
 <layer number="1" name="Top" color="4" fill="1" visible="yes" active="yes"/>
@@
 <wire x1="22.86" y1="77.47" x2="0" y2="77.47" width="0" layer="20"/>
 <wire x1="0" y1="77.47" x2="0" y2="-1.27" width="0" layer="20"/>
-<text x="13.462" y="1625.6" size="1.27" layer="25" align="center">-</text>
 <hole x="19.05" y="73.66" drill="2.8"/>
 <circle x="19.05" y="73.66" radius="1.778" width="1.905" layer="42"/>
@@
 <via x="10.16" y="51.562" extent="1-16" drill="0.5"/>
 <via x="20.955" y="16.51" extent="1-16" drill="0.5"/>
-<wire x1="3.81" y1="29.075" x2="3.81" y2="31.242" width="0.4064" layer="16"/>
 <via x="3.81" y="31.242" extent="1-16" drill="0.5"/>
 <wire x1="5.08" y1="17.82" x2="3.81" y2="16.55" width="0.4064" layer="1"/>
@@
 <wire x1="5.207" y1="24.704" x2="5.08" y2="24.577" width="0.4064" layer="1"/>
 <wire x1="5.08" y1="24.577" x2="5.08" y2="22.86" width="0.4064" layer="1"/>
+<wire x1="3.81" y1="31.242" x2="3.81" y2="29.45" width="0.4064" layer="16"/>
 <wire x1="6.35" y1="68.11" x2="6.35" y2="66.51" width="0" layer="19" extent="1-1"/>
-<wire x1="3.81" y1="29.45" x2="3.81" y2="29.075" width="0" layer="19" extent="16-16"/>
 <wire x1="2.54" y1="64.77" x2="6.35" y2="64.77" width="0" layer="19" extent="1-1"/>
 </signal>
@@
 <wire x1="13.335" y1="31.115" x2="13.335" y2="28.575" width="0.4064" layer="1"/>
 <via x="13.335" y="28.575" extent="1-16" drill="0.6"/>
-<wire x1="8.89" y1="27.94" x2="7.62" y2="29.21" width="0.4064" layer="1"/>
-<wire x1="7.62" y1="29.21" x2="7.62" y2="31.75" width="0.4064" layer="1"/>
-<wire x1="7.62" y1="31.75" x2="6.35" y2="33.02" width="0.4064" layer="1"/>
 <wire x1="6.35" y1="33.02" x2="6.35" y2="38.1" width="0.4064" layer="1"/>
 <via x="6.35" y="38.1" extent="1-16" drill="0.6"/>
 <wire x1="5.207" y1="26.604" x2="5.273" y2="26.67" width="0.4064" layer="1"/>
-<wire x1="5.273" y1="26.67" x2="7.62" y2="27.432" width="0.4064" layer="1"/>
-<wire x1="7.62" y1="27.432" x2="8.89" y2="27.94" width="0.4064" layer="1"/>
-<wire x1="3.81" y1="26.67" x2="3.81" y2="28.2" width="0" layer="19" extent="1-16"/>
+<wire x1="6.35" y1="33.02" x2="8.89" y2="30.48" width="0.4064" layer="1"/>
+<wire x1="8.89" y1="30.48" x2="8.89" y2="27.94" width="0.4064" layer="1"/>
+<wire x1="5.776" y1="26.604" x2="5.207" y2="26.604" width="0.4064" layer="1"/>
+<wire x1="5.776" y1="26.604" x2="6.223" y2="27.051" width="0.4064" layer="1"/>
+<wire x1="6.223" y1="27.051" x2="8.128" y2="27.051" width="0.4064" layer="1"/>
+<wire x1="8.128" y1="27.051" x2="8.89" y2="27.813" width="0.4064" layer="1"/>
+<wire x1="8.89" y1="27.813" x2="8.89" y2="27.94" width="0.4064" layer="1"/>
 </signal>
 <signal name="RESET">
@@
 <wire x1="3.81" y1="24.45" x2="2.22" y2="24.45" width="0.4064" layer="16"/>
 <wire x1="2.22" y1="24.45" x2="1.27" y2="25.4" width="0.4064" layer="16"/>
-<wire x1="1.27" y1="25.4" x2="1.27" y2="31.75" width="0.4064" layer="16"/>
 <wire x1="1.27" y1="31.75" x2="3.81" y2="34.29" width="0.4064" layer="16"/>
+<wire x1="1.27" y1="31.75" x2="1.27" y2="25.4" width="0.4064" layer="16"/>
 </signal>
 <signal name="N$4">
@@
 <wire x1="4.318" y1="65.786" x2="1.27" y2="62.738" width="0.4064" layer="16"/>
 <via x="2.54" y="35.56" extent="1-16" drill="0.5"/>
-<wire x1="3.81" y1="26.95" x2="5.36" y2="26.95" width="0.4064" layer="16"/>
-<wire x1="5.36" y1="26.95" x2="6.604" y2="28.575" width="0.4064" layer="16"/>
-<via x="6.604" y="28.575" extent="1-16" drill="0.6"/>
-<wire x1="6.604" y1="28.575" x2="6.604" y2="31.115" width="0.4064" layer="1"/>
-<wire x1="6.604" y1="31.115" x2="2.54" y2="35.56" width="0.4064" layer="1"/>
+<wire x1="3.81" y1="26.95" x2="5.995" y2="26.95" width="0.4064" layer="16"/>
+<via x="7.366" y="28.067" extent="1-16" drill="0.6"/>
+<wire x1="7.366" y1="28.067" x2="7.366" y2="30.099" width="0.4064" layer="1"/>
+<wire x1="7.366" y1="30.099" x2="2.54" y2="35.56" width="0.4064" layer="1"/>
 <wire x1="2.54" y1="35.56" x2="1.27" y2="36.83" width="0.4064" layer="16"/>
 <wire x1="1.27" y1="36.83" x2="1.27" y2="62.738" width="0.4064" layer="16"/>
+<wire x1="7.366" y1="28.067" x2="5.995" y2="26.95" width="0.4064" layer="16"/>
 </signal>
 <signal name="RX">

Commit message: Updated circuit shematic to reflect current working board version
Parts:
- R3: value 50k -> 50 kOhm
- R4, R5, R6: value 150 -> 150 Ohm
Changed lines of the file:
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@@
 <?xml version="1.0" encoding="utf-8"?>
 <!DOCTYPE eagle SYSTEM "eagle.dtd">
-<eagle version="7.6.0">
+<eagle version="7.5.0">
 <drawing>
 <settings>
@@
 <attribute name="NAME" x="17.621" y="8.509" size="0.762" layer="25" rot="R90"/>
 </element>
-<element name="R3" library="rcl" package="R0603" value="50k" x="14.83868125" y="34.556696875" smashed="yes" rot="MR270">
+<element name="R3" library="rcl" package="R0603" value="50 kOhm" x="14.83868125" y="34.556696875" smashed="yes" rot="MR270">
 <attribute name="VALUE" x="14.408815625" y="37.88576875" size="0.762" layer="28" rot="MR225"/>
 </element>
-<element name="R4" library="resistor" package="R0402" value="150" x="18.51" y="12.6365" smashed="yes" rot="R90"/>
+<element name="R4" library="resistor" package="R0402" value="150 Ohm" x="18.51" y="12.6365" smashed="yes" rot="R90"/>
 <element name="RESET" library="pinhead" package="1X02" value="" x="18.542" y="36.322" smashed="yes">
 <attribute name="NAME" x="22.24188125" y="34.41690625" size="1.27" layer="25" ratio="10" rot="R180"/>
@@
 <attribute name="VALUE" x="15.24" y="44.577" size="1.27" layer="28" ratio="10" rot="MR0"/>
 </element>
-<element name="R5" library="resistor" package="R0402" value="150" x="5.588" y="52.832" smashed="yes" rot="MR270">
+<element name="R5" library="resistor" package="R0402" value="150 Ohm" x="5.588" y="52.832" smashed="yes" rot="MR270">
 <attribute name="VALUE" x="7.747" y="54.229" size="1.27" layer="28" rot="MR270"/>
 </element>
-<element name="R6" library="resistor" package="R0402" value="150" x="11.938" y="38.1" smashed="yes" rot="MR0"/>
+<element name="R6" library="resistor" package="R0402" value="150 Ohm" x="11.938" y="38.1" smashed="yes" rot="MR0"/>
 <element name="YAW" library="Random" package="35RA_SMT" value="3.5MMJACK" x="22.86" y="57.15" rot="R180"/>
 <element name="MOTPWR" library="pinhead" package="1X02" value="" x="7.62" y="72.39" smashed="yes" rot="R270">
